File: hardware/rom-programmer.kicad_sch (KiCad schematic)
At the start: 19 parts, among them U1 74HC595, U2 74HC595, U3 28C256

Commit message: Added schematic PDF
Other:
- title: 28Cxxx EEROM Programmer -> 28Cx EEROM Programmer
Changed lines of the file:
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@@
 	(paper "A4")
 	(title_block
-		(title "28Cxxx EEROM Programmer")
-		(rev "0")
+		(title "28Cx EEROM Programmer")
+		(rev "A")
 		(company "The Network Entropologist")
 	)
