File: hardware/rom-programmer.kicad_sch (KiCad schematic)
At the start: 19 parts, among them U1 74HC595, U2 74HC595, U3 28C256

Commit message: Checkpoint
Connections:
- net ~{ROM_CE}: now also A1.21 (A2); no longer A1.20 (A1)
- net ~{ROM_OE}: now also A1.20 (A1); no longer A1.16 (D13)
- net ~{ROM_WE}: now also A1.19 (A0); no longer A1.21 (A2)
- net ~{SEROE}: now also A1.23 (A4); no longer A1.22 (A3)
- net ~{SRCLR}: now also A1.22 (A3); no longer A1.19 (A0)
