File: hardware/rom-programmer.kicad_sch (KiCad schematic)
At the start: 19 parts, among them U1 74HC595, U2 74HC595, U3 28C256

Commit message: Writing files works
Parts:
- C1, C6, C9: value 1uF -> 2.2uF
Connections:
- net CRCLR is gone; now on net ~{SRCLR}: U1.10 (~{SRCLR}), U2.10 (~{SRCLR})
- net ~{SER_OE} is gone; now on net ~{SEROE}: U1.13 (~{OE}), U2.13 (~{OE})
Other:
- moved on the sheet: A1, C1, C10, C11, C2, C3, C4, C5, C6, C7, C8, C9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
