File: hardware-pth/rom-programmer.kicad_pcb (KiCad board)
At the start: 2 copper layers, 120 x 70 mm, 21 parts, among them U1 74HC595, U2 74HC595, U3 28C256

Commit message: Can now read a single byte from the CLI
Parts:
- moved REF** 81.9 mm to (190.5, 115.5)
- moved G*** 61.0 mm to (136.5, 71.3)
- moved H2 11.0 mm to (193.0, 60.5)
- moved H3 11.0 mm to (193.0, 124.5)
Connections:
- U1 pad 10: /CRCLR -> /~{SRCLR}
- U1 pad 13: /~{SER_OE} -> /~{SEROE}
- U2 pad 10: /CRCLR -> /~{SRCLR}
- U2 pad 13: /~{SER_OE} -> /~{SEROE}
Routing:
- net /~{SRCLR}: track 0.00 -> 184.0 mm, vias 0 -> 2
- net /~{SEROE}: track 0.00 -> 171.0 mm, vias 0 -> 2
- net /RCLK: track 58.0 -> 171.2 mm, vias 3 -> 0
- net /SRCLK: track 63.3 -> 166.8 mm, vias 3 -> 4
- net /SERO: track 3.79 -> 101.0 mm, vias 1 -> 4
- net /~{ROM_WE}: track 0.00 -> 91.7 mm
- net /~{ROM_OE}: track 0.00 -> 78.7 mm
- net /~{ROM_CE}: track 0.00 -> 74.0 mm
- net /A12: track 37.1 -> 50.1 mm, vias 1 -> 2
- net /A14: track 41.0 -> 53.8 mm, vias 1 -> 2
- net /~{SER_OE}: track 8.86 -> 0.00 mm, vias 2 -> 0
- net /SRDATA: track 54.7 -> 51.4 mm
- net /CRCLR: track 2.68 -> 0.00 mm, vias 1 -> 0
- net GND: track 0.00 -> 2.19 mm, vias 0 -> 70
- net /A13: track 22.6 -> 24.4 mm
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Other:
- board size 120 x 70 mm -> 109 x 70 mm
